File: boards/controller_board/KPMC_brug_controller.sch (KiCad schematic (older format))
At the start: 23 parts, among them J1 Screw_Terminal_1x02, J2 Screw_Terminal_1x02, P1 CONN_01X04, P2 CONN_01X08, U1 LM7805CT

Commit message: add display backlight blinky
Parts:
- removed C7: 1uF, symbol C
- removed RV1: POT_TRIM, symbol POT_TRIM
- added C11, C12, C13, C14: 100nF, symbol C
- added P3, P4: CONN_01X02, symbol CONN_01X02
- added P5, P6, P7: CONN_01X03, symbol CONN_01X03
- added P8, P9: CONN_01X04, symbol CONN_01X04
- added R3, R4: 1k, symbol R
- C1: footprint (none) -> Capacitors_THT:CP_Radial_D17.0mm_P7.50mm
- C2, C4: footprint (none) -> Capacitors_THT:C_Rect_L7.2mm_W2.5mm_P5.00mm_FKS2_FKP2_MKS2_MKP2
- C3: footprint (none) -> Capacitors_THT:CP_Axial_L30.0mm_D10.0mm_P35.00mm_Horizontal
- C5: footprint (none) -> Capacitors_THT:C_Axial_L5.1mm_D3.1mm_P7.50mm_Horizontal
- C7: renamed from C?; footprint (none) -> Capacitors_THT:CP_Radial_D17.0mm_P7.50mm
- gave numbers to parts that had none: 4
Connections:
- wire segments 38 -> 134
Other:
- note added: "6050"
- note added: "LCD"
- note added: "MOTOR L298 EN,In1, In2"
- note added: "Nav lichten B"
- note added: "RX 433MHz module"
- note added: "Slagbomen"
- note added: "nav lichten A"
